Commit message: Update robot_core.xacro
changing chassis and adding rear left wheel

File: description/robot_core.xacro (robot description, xacro)
@@ -1,5 +1,5 @@
 <?xml version="1.0"?>
 <robot xmlns:xacro="http://www.ros.org/wiki/xacro" >
-    <xacro:include filename="inertial_macros.xacro"/>
+    <!-- <xacro:include filename="inertial_macros.xacro"/> -->
     <material name="white">
         <color rgba="1 1 1 1" />
@@ -28,101 +28,26 @@
     <link name="chassis">
         <visual>
-            <origin xyz="0.15 0 0.075"/>
+            <origin xyz="0.055 0 0.0485"/>
             <geometry>
-                <box size="0.3 0.3 0.15"/>
+                <box size="0.515 0.31 0.135"/>
+                <!-- l bh -->
             </geometry>
             <material name="white"/>
         </visual>
-        <collision>
-            <origin xyz="0.15 0 0.075"/>
-            <geometry>
-                <box size="0.3 0.3 0.15"/>
-            </geometry>
-        </collision>
-        <xacro:inertial_box mass="0.5" x="0.3" y="0.3" z="0.15">
-            <origin xyz="0.15 0 0.075" rpy="0 0 0"/>
-        </xacro:inertial_box>
     </link>
-    <gazebo reference="chassis">
-        <material>Gazebo/White</material>
-    </gazebo>
-    <!-- LEFT WHEEL LINK -->
-    <joint name="left_wheel_joint" type="continuous">
-        <parent link="base_link"/>
-        <child link="left_wheel"/>
-        <origin xyz="0 0.175 0" rpy="-${pi/2} 0 0" />
-        <axis xyz="0 0 1"/>
-    </joint>
-    <link name="left_wheel">
-        <visual>
-            <geometry>
-                <cylinder radius="0.05" length="0.04"/>
-            </geometry>
-            <material name="blue"/>
-        </visual>
-        <collision>
-            <geometry>
-                <cylinder radius="0.05" length="0.04"/>
-            </geometry>
-        </collision>
-        <xacro:inertial_cylinder mass="0.1" length="0.04" radius="0.05">
-            <origin xyz="0 0 0" rpy="0 0 0"/>
-        </xacro:inertial_cylinder>
-    </link>
-    <gazebo reference="left_wheel">
-        <material>Gazebo/Blue</material>
-    </gazebo>
-    <!-- RIGHT WHEEL LINK -->
-    <joint name="right_wheel_joint" type="continuous">
-        <parent link="base_link"/>
-        <child link="right_wheel"/>
-        <origin xyz="0 -0.175 0" rpy="${pi/2} 0 0" />
-        <axis xyz="0 0 -1"/>
-    </joint>
-    <link name="right_wheel">
-        <visual>
-            <geometry>
-                <cylinder radius="0.05" length="0.04"/>
-            </geometry>
-            <material name="blue"/>
-        </visual>
-        <collision>
-            <geometry>
-                <cylinder radius="0.05" length="0.04"/>
-            </geometry>
-        </collision>
-        <xacro:inertial_cylinder mass="0.1" length="0.04" radius="0.05">
-            <origin xyz="0 0 0" rpy="0 0 0"/>
-        </xacro:inertial_cylinder>
-    </link>
-    <gazebo reference="right_wheel">
-        <material>Gazebo/Blue</material>
-    </gazebo>
-    <!-- CASTER WHEEL LINK -->
-    <joint name="caster_wheel_joint" type="fixed">
-        <parent link="chassis"/>
-        <child link="caster_wheel"/>
-        <origin xyz="0.24 0 0"/>
-    </joint>
-    <link name="caster_wheel">
-        <visual>
-            <geometry>
-                <sphere radius="0.05"/>
-            </geometry>
-            <material name="black"/>
-        </visual>
-        <collision>
-            <geometry>
-                <sphere radius="0.05"/>
-            </geometry>
-        </collision>
-        <xacro:inertial_sphere mass="0.1" radius="0.05">
-            <origin xyz="0 0 0" rpy="0 0 0"/>
-        </xacro:inertial_sphere>
-    </link>
-    <gazebo reference="caster_wheel">
-        <material>Gazebo/Black</material>
-        <mu1 value="0.001"/>
-        <mu2 value="0.002"/>
-    </gazebo>
-</robot>
+  <!-- Rear LEFT WHEEL -->
+<joint name="rear_left_wheel_joint" type="continuous">
+    <parent link="base_link"/>
+    <child link="rear_left_wheel"/>
+    <origin xyz="0 0.155 0" rpy="-${pi/2} 0 0"/>
+    <axis xyz="0 0 1"/>
+</joint>
+<link name="rear_left_wheel">
+    <visual>
+        <geometry>
+            <cylinder length="0.04" radius="0.0485" />
+        </geometry>
+        <material name="blue"/>
+    </visual>
+</link>
+    </robot>

Commit message: modified:   description/robot_core.xacro

File: description/robot_core.xacro (robot description, xacro)
@@ -54,2 +54,20 @@
 </link>
     </robot>
+  <!-- Rear right WHEEL -->
+<joint name="rear_right_wheel_joint" type="continuous">
+    <parent link="base_link"/>
+    <child link="rear_right_wheel"/>
+    <origin xyz="0 -0.18 0" rpy="-${pi/2} 0 0"/>
+    <!-- y = b + thickness of wheel/2 + 0.5(mm) -->
+    <!-- connected with base link -->
+    <axis xyz="0 0 -1"/>
+</joint>
+<link name="rear_right_wheel">
+    <visual>
+        <geometry>
+            <cylinder length="0.04" radius="0.0485" />
+        </geometry>
+        <material name="blue"/>
+    </visual>
+</link>
+    </robot>

Commit message: modified:   description/robot_core.xacro

File: description/robot_core.xacro (robot description, xacro)
@@ -17,5 +17,5 @@
         <color rgba="1 0 0 1"/>
     </material>
-    <!-- BASE LINK -->
+    <!-- REAR BASE LINK -->
     <link name="base_link">
     </link>
@@ -53,6 +53,5 @@
     </visual>
 </link>
-    </robot>
-  <!-- Rear right WHEEL -->
+  <!-- Rear RIGHT WHEEL -->
 <joint name="rear_right_wheel_joint" type="continuous">
     <parent link="base_link"/>
@@ -71,3 +70,42 @@
     </visual>
 </link>
+<!-- FRONT -->
+    <!-- FRONT BASE LINK -->
+    <link name="base2_link">
+            <origin xyz="0.360 0 0"/>
+    </link>
+  <!-- FRONT LEFT WHEEL -->
+<joint name="front_left_wheel_joint" type="continuous">
+    <parent link="base2_link"/>
+    <child link="front_left_wheel"/>
+    <origin xyz="0.360 0.18 0" rpy="-${pi/2} 0 0"/>
+    <!-- y = b + thickness of wheel/2 + 0.5(mm) -->
+    <!-- connected with base link -->
+    <axis xyz="0 0 1"/>
+</joint>
+<link name="front_left_wheel">
+    <visual>
+        <geometry>
+            <cylinder length="0.04" radius="0.0485" />
+        </geometry>
+        <material name="blue"/>
+    </visual>
+</link>
+  <!-- FRONT RIGHT WHEEL -->
+<joint name="front_right_wheel_joint" type="continuous">
+    <parent link="base2_link"/>
+    <child link="front_left_wheel"/>
+    <origin xyz="0.360 -0.18 0" rpy="-${pi/2} 0 0"/>
+    <!-- y = b + thickness of wheel/2 + 0.5(mm) -->
+    <!-- connected with base link -->
+    <axis xyz="0 0 -1"/>
+</joint>
+<link name="front_right_wheel">
+    <visual>
+        <geometry>
+            <cylinder length="0.04" radius="0.0485" />
+        </geometry>
+        <material name="blue"/>
+    </visual>
+</link>
     </robot>

Commit message: modified:   description/robot_core.xacro

File: description/robot_core.xacro (robot description, xacro)
@@ -72,7 +72,12 @@
 <!-- FRONT -->
     <!-- FRONT BASE LINK -->
-    <link name="base2_link">
-            <origin xyz="0.360 0 0"/>
-    </link>
+<joint name="base2_joint" type="continuous">
+    <parent link="base_link"/>
+    <child link="base2_link"/>
+    <origin xyz="0.360 0 0"/>
+    <limit effort="1000.0" lower="0.0" upper="0.548" velocity="0.5"/>
+</joint>
+<link name="base2_ link">
+</link>
   <!-- FRONT LEFT WHEEL -->
 <joint name="front_left_wheel_joint" type="continuous">

Commit message: modified:   description/robot_core.xacro

File: description/robot_core.xacro (robot description, xacro)
@@ -71,13 +71,4 @@
 </link>
 <!-- FRONT -->
-    <!-- FRONT BASE LINK -->
-<joint name="base2_joint" type="continuous">
-    <parent link="base_link"/>
-    <child link="base2_link"/>
-    <origin xyz="0.360 0 0"/>
-    <limit effort="1000.0" lower="0.0" upper="0.548" velocity="0.5"/>
-</joint>
-<link name="base2_ link">
-</link>
   <!-- FRONT LEFT WHEEL -->
 <joint name="front_left_wheel_joint" type="continuous">
@@ -97,4 +88,19 @@
     </visual>
 </link>
+<joint name="front_left_wheel_steer_joint" type="revolute">
+    <limit lower="-1" upper="1" effort="1" velocity="5"/>
+    <axis xyz="0 0 1"/>
+    <parent link="base_link"/>
+    <child link="front_left_wheel_steer"/>
+    <origin rpy="0 0 0" xyz="0.360 0.18 0"/>
+  </joint>
+<link name="front_left_wheel_steer">
+    <visual>
+      <geometry>
+        <cylinder length="0.01" radius="0.01"/>
+      </geometry>
+      <material name="black"/>
+    </visual>
+  </link>
   <!-- FRONT RIGHT WHEEL -->
 <joint name="front_right_wheel_joint" type="continuous">
@@ -114,3 +120,18 @@
     </visual>
 </link>
+<joint name="front_right_wheel_steer_joint" type="revolute">
+    <limit lower="-1" upper="1" effort="1" velocity="5"/>
+    <axis xyz="0 0 1"/>
+    <parent link="base_link"/>
+    <child link="front_right_wheel_steer"/>
+    <origin rpy="0 0 0" xyz="0.360 -0.18 0"/>
+  </joint>
+<link name="front_right_wheel_steer">
+    <visual>
+      <geometry>
+        <cylinder length="0.01" radius="0.01"/>
+      </geometry>
+      <material name="black"/>
+    </visual>
+  </link>
     </robot>

Commit message: modified:   description/robot_core.xacro

File: description/robot_core.xacro (robot description, xacro)
@@ -73,5 +73,5 @@
   <!-- FRONT LEFT WHEEL -->
 <joint name="front_left_wheel_joint" type="continuous">
-    <parent link="base2_link"/>
+    <parent link="front_left_wheel_steer"/>
     <child link="front_left_wheel"/>
     <origin xyz="0.360 0.18 0" rpy="-${pi/2} 0 0"/>
@@ -105,5 +105,5 @@
   <!-- FRONT RIGHT WHEEL -->
 <joint name="front_right_wheel_joint" type="continuous">
-    <parent link="base2_link"/>
+    <parent link="front_right_wheel_steer"/>
     <child link="front_left_wheel"/>
     <origin xyz="0.360 -0.18 0" rpy="-${pi/2} 0 0"/>

Commit message: Update robot_core.xacro

File: description/robot_core.xacro (robot description, xacro)
@@ -106,5 +106,5 @@
 <joint name="front_right_wheel_joint" type="continuous">
     <parent link="front_right_wheel_steer"/>
-    <child link="front_left_wheel"/>
+    <child link="front_right_wheel"/>
     <origin xyz="0.360 -0.18 0" rpy="-${pi/2} 0 0"/>
     <!-- y = b + thickness of wheel/2 + 0.5(mm) -->
