Commit message: modified:   description/robot.urdf.xacro 	modified:   description/robot_core.xacro

File: description/robot.urdf.xacro (robot description, xacro)
@@ -2,6 +2,6 @@
 <robot xmlns:xacro="http://www.ros.org/wiki/xacro"  name="robot">
 <xacro:include filename="robot_core.xacro" />
-<xacro:include filename="gazebo_control.xacro" />
-<xacro:include filename="lidar.xacro" />
-<xacro:include filename="camera.xacro" />
+<!-- <xacro:include filename="gazebo_control.xacro" /> -->
+<!-- <xacro:include filename="lidar.xacro" /> -->
+<!-- <xacro:include filename="camera.xacro" /> -->
 </robot>

File: description/robot_core.xacro (robot description, xacro)
@@ -28,8 +28,8 @@
     <link name="chassis">
         <visual>
-            <origin xyz="0.055 0 0.0485"/>
+            <origin xyz="0.2575 0 0.0675"/>
             <geometry>
                 <box size="0.515 0.31 0.135"/>
-                <!-- l bh -->
+                <!-- l b h -->
             </geometry>
             <material name="white"/>
@@ -40,5 +40,7 @@
     <parent link="base_link"/>
     <child link="rear_left_wheel"/>
-    <origin xyz="0 0.155 0" rpy="-${pi/2} 0 0"/>
+    <origin xyz="0 0.18 0" rpy="-${pi/2} 0 0"/>
+    <!-- y = b + thickness of wheel/2 + 0.5(mm) -->
+    <!-- connected with base link -->
     <axis xyz="0 0 1"/>
 </joint>

Commit message: modified:   description/robot.urdf.xacro 	modified:   description/robot_core2.xacro

File: description/robot.urdf.xacro (robot description, xacro)
@@ -1,5 +1,6 @@
 <?xml version="1.0"?>
 <robot xmlns:xacro="http://www.ros.org/wiki/xacro"  name="robot">
-<xacro:include filename="robot_core.xacro" />
+<xacro:include filename="robot_core2.xacro" />
+<!-- <xacro:include filename="robot_core.xacro" /> -->
 <!-- <xacro:include filename="gazebo_control.xacro" /> -->
 <!-- <xacro:include filename="lidar.xacro" /> -->

File: description/robot_core2.xacro (robot description, xacro)
@@ -30,5 +30,5 @@
             <origin xyz="0.2575 0 0.0675"/>
             <geometry>
-                <box size="0.515 0.31 0.135"/>
+                <box size="0.515 0.31 0.097"/>
                 <!-- l b h -->
             </geometry>
@@ -49,16 +49,16 @@
     </gazebo> -->
     <!-- UPPER CHASSIS LINK -->
-<joint name="chassis_joint" type="fixed">
+<joint name="upper_chassis_joint" type="fixed">
     <parent link="chassis"/>
     <child link="upper_chassis"/>
-    <origin xyz="0.2575 0 0.0675"/>
+    <origin xyz="0.235 0 0.097"/>
 </joint>
 <link name="upper_chassis">
     <visual>
-        <origin xyz="0.2575 0.097 0.0675" rpy="0 0 0"/>
+        <origin xyz="0 0 0.038" rpy="0 0 0"/>
         <geometry>
-            <box size="0.263 0.31 0.038"/>
+            <box size="0.263 0.31 0.04"/>
         </geometry>
-        <material name="white"/>
+        <material name="red"/>
     </visual>
 </link>
@@ -67,5 +67,5 @@
     <parent link="base_link"/>
     <child link="rear_left_wheel"/>
-    <origin xyz="0 0.18 0" rpy="-${pi/2} 0 0"/>
+    <origin xyz="0 0.18 0.0194" rpy="-${pi/2} 0 0"/>
     <!-- y = b + thickness of wheel/2 + 0.5(mm) -->
     <!-- connected with base link -->
@@ -84,5 +84,5 @@
     <parent link="base_link"/>
     <child link="rear_right_wheel"/>
-    <origin xyz="0 -0.18 0" rpy="-${pi/2} 0 0"/>
+    <origin xyz="0 -0.18 0.0194" rpy="-${pi/2} 0 0"/>
     <!-- y = b + thickness of wheel/2 + 0.5(mm) -->
     <!-- connected with base link -->
@@ -117,5 +117,5 @@
     <parent link="front_wheel_steer"/>
     <child link="front_left_wheel"/>
-    <origin xyz="0 0.18 0" rpy="-${pi/2} 0 0"/>
+    <origin xyz="0 0.18 0.0194" rpy="-${pi/2} 0 0"/>
     <!-- y = b + thickness of wheel/2 + 0.5(mm) -->
     <!-- connected with base link -->
@@ -134,5 +134,5 @@
     <parent link="front_wheel_steer"/>
     <child link="front_right_wheel"/>
-    <origin xyz="0 -0.18 0" rpy="-${pi/2} 0 0"/>
+    <origin xyz="0 -0.18 0.0194" rpy="-${pi/2} 0 0"/>
     <!-- y = b + thickness of wheel/2 + 0.5(mm) -->
     <!-- connected with base link -->
