Commit message: modified:   description/robot_core2.xacro

File: description/robot_core2.xacro (robot description, xacro)
@@ -76,5 +76,5 @@
     <parent link="base_link"/>
     <child link="front_wheel_steer"/>
-    <origin rpy="0 0 0" xyz="0.360 0.18 0"/>
+    <origin rpy="0 0 0" xyz="0.360 0 0"/>
   </joint>
 <link name="front_wheel_steer">
@@ -90,5 +90,5 @@
     <parent link="front_wheel_steer"/>
     <child link="front_left_wheel"/>
-    <origin xyz="0.360 0.18 0" rpy="-${pi/2} 0 0"/>
+    <origin xyz="0 0.18 0" rpy="-${pi/2} 0 0"/>
     <!-- y = b + thickness of wheel/2 + 0.5(mm) -->
     <!-- connected with base link -->
@@ -103,25 +103,9 @@
     </visual>
 </link>
-<!--
-<joint name="front_left_wheel_steer_joint" type="revolute">
-    <limit lower="-1" upper="1" effort="1" velocity="5"/>
-    <axis xyz="0 0 1"/>
-    <parent link="base_link"/>
-    <child link="front_left_wheel_steer"/>
-    <origin rpy="0 0 0" xyz="0.360 0.18 0"/>
-  </joint>
-<link name="front_left_wheel_steer">
-    <visual>
-      <geometry>
-        <cylinder length="0.01" radius="0.01"/>
-      </geometry>
-      <material name="black"/>
-    </visual>
-  </link>  -->
   <!-- FRONT RIGHT WHEEL -->
 <joint name="front_right_wheel_joint" type="continuous">
     <parent link="front_wheel_steer"/>
     <child link="front_right_wheel"/>
-    <origin xyz="0.360 -0.18 0" rpy="-${pi/2} 0 0"/>
+    <origin xyz="0 -0.18 0" rpy="-${pi/2} 0 0"/>
     <!-- y = b + thickness of wheel/2 + 0.5(mm) -->
     <!-- connected with base link -->
@@ -136,18 +120,3 @@
     </visual>
 </link>
-<!-- <joint name="front_right_wheel_steer_joint" type="revolute">
-    <limit lower="-1" upper="1" effort="1" velocity="5"/>
-    <axis xyz="0 0 1"/>
-    <parent link="base_link"/>
-    <child link="front_right_wheel_steer"/>
-    <origin rpy="0 0 0" xyz="0.360 -0.18 0"/>
-  </joint>
-<link name="front_right_wheel_steer">
-    <visual>
-      <geometry>
-        <cylinder length="0.01" radius="0.01"/>
-      </geometry>
-      <material name="black"/>
-    </visual>
-  </link>  -->
     </robot>

Commit message: modified:   description/robot_core2.xacro

File: description/robot_core2.xacro (robot description, xacro)
@@ -35,5 +35,17 @@
             <material name="white"/>
         </visual>
+        <collision>
+            <origin xyz="0.2575 0 0.0675"/>
+            <geometry>
+                <box size="0.515 0.31 0.135"/>
+            </geometry>
+        </collision>
+        <xacro:inertial_box mass="0.5" x="0.515" y="0.31" z="0.135">
+            <origin xyz="0.2575 0 0.0675" rpy="0 0 0"/>
+        </xacro:inertial_box>
     </link>
+    <gazebo reference="chassis">
+        <material>Gazebo/White</material>
+    </gazebo>
   <!-- Rear LEFT WHEEL -->
 <joint name="rear_left_wheel_joint" type="continuous">

Commit message: modified:   description/robot_core2.xacro

File: description/robot_core2.xacro (robot description, xacro)
@@ -35,5 +35,5 @@
             <material name="white"/>
         </visual>
-        <collision>
+        <!-- <collision>
             <origin xyz="0.2575 0 0.0675"/>
             <geometry>
@@ -43,9 +43,24 @@
         <xacro:inertial_box mass="0.5" x="0.515" y="0.31" z="0.135">
             <origin xyz="0.2575 0 0.0675" rpy="0 0 0"/>
-        </xacro:inertial_box>
+        </xacro:inertial_box>   -->
     </link>
-    <gazebo reference="chassis">
+    <!-- <gazebo reference="chassis">
         <material>Gazebo/White</material>
-    </gazebo>
+    </gazebo> -->
+    <!-- UPPER CHASSIS LINK -->
+<joint name="chassis_joint" type="fixed">
+    <parent link="chassis"/>
+    <child link="upper_chassis"/>
+    <origin xyz="0.2575 0 0.0675"/>
+</joint>
+<link name="upper_chassis">
+    <visual>
+        <origin xyz="0.2575 0.097 0.0675" rpy="0 0 0"/>
+        <geometry>
+            <box size="0.263 0.31 0.038"/>
+        </geometry>
+        <material name="white"/>
+    </visual>
+</link>
   <!-- Rear LEFT WHEEL -->
 <joint name="rear_left_wheel_joint" type="continuous">

Commit message: Update robot_core2.xacro

File: description/robot_core2.xacro (robot description, xacro)
@@ -56,5 +56,9 @@
 <link name="upper_chassis">
     <visual>
+<<<<<<< HEAD
+        <origin xyz="0.2575 0 0.097" rpy="0 0 0"/>
+=======
         <origin xyz="0 0 0.038" rpy="0 0 0"/>
+>>>>>>> 6796d58cfbd689a60f0606a5cd9eb66f05d851cd
         <geometry>
             <box size="0.263 0.31 0.04"/>
@@ -98,5 +102,5 @@
 </link>
 <!-- FRONT -->
-<joint name="front_wheel_steer_joint" type="revolute">
+<!-- <joint name="front_wheel_steer_joint" type="revolute">
     <limit lower="-1" upper="1" effort="1" velocity="5"/>
     <axis xyz="0 0 1"/>
@@ -112,8 +116,8 @@
       <material name="black"/>
     </visual>
-  </link>
+  </link>  -->
   <!-- FRONT LEFT WHEEL -->
 <joint name="front_left_wheel_joint" type="continuous">
-    <parent link="front_wheel_steer"/>
+    <parent link="front_left_wheel_steer"/>
     <child link="front_left_wheel"/>
     <origin xyz="0 0.18 0.0194" rpy="-${pi/2} 0 0"/>
@@ -130,7 +134,22 @@
     </visual>
 </link>
+<joint name="front_left_wheel_steer_joint" type="revolute">
+    <limit lower="-1" upper="1" effort="1" velocity="5"/>
+    <axis xyz="0 0 1"/>
+    <parent link="base_link"/>
+    <child link="front__left_wheel_steer"/>
+    <origin rpy="0 0 0" xyz="0.360 0 0"/>
+  </joint>
+<link name="front_left_wheel_steer">
+    <visual>
+      <geometry>
+        <cylinder length="0.01" radius="0.01"/>
+      </geometry>
+      <material name="black"/>
+    </visual>
+  </link>
   <!-- FRONT RIGHT WHEEL -->
 <joint name="front_right_wheel_joint" type="continuous">
-    <parent link="front_wheel_steer"/>
+    <parent link="front_right_wheel_steer"/>
     <child link="front_right_wheel"/>
     <origin xyz="0 -0.18 0.0194" rpy="-${pi/2} 0 0"/>
@@ -147,3 +166,18 @@
     </visual>
 </link>
+<joint name="front_right_wheel_steer_joint" type="revolute">
+    <limit lower="-1" upper="1" effort="1" velocity="5"/>
+    <axis xyz="0 0 1"/>
+    <parent link="base_link"/>
+    <child link="front_right_wheel_steer"/>
+    <origin rpy="0 0 0" xyz="0.360 0 0"/>
+  </joint>
+<link name="front_right_wheel_steer">
+    <visual>
+      <geometry>
+        <cylinder length="0.01" radius="0.01"/>
+      </geometry>
+      <material name="black"/>
+    </visual>
+  </link>
     </robot>

Commit message: Update robot_core2.xacro

File: description/robot_core2.xacro (robot description, xacro)
@@ -35,13 +35,11 @@
             <material name="white"/>
         </visual>
-        <!-- <collision>
+        <collision>
             <origin xyz="0.2575 0 0.0675"/>
             <geometry>
-                <box size="0.515 0.31 0.135"/>
+                <box size="0.515 0.31 0.097"/>
+                <!-- l b h -->
             </geometry>
         </collision>
-        <xacro:inertial_box mass="0.5" x="0.515" y="0.31" z="0.135">
-            <origin xyz="0.2575 0 0.0675" rpy="0 0 0"/>
-        </xacro:inertial_box>   -->
     </link>
     <!-- <gazebo reference="chassis">
@@ -56,9 +54,5 @@
 <link name="upper_chassis">
     <visual>
-<<<<<<< HEAD
-        <origin xyz="0.2575 0 0.097" rpy="0 0 0"/>
-=======
         <origin xyz="0 0 0.038" rpy="0 0 0"/>
->>>>>>> 6796d58cfbd689a60f0606a5cd9eb66f05d851cd
         <geometry>
             <box size="0.263 0.31 0.04"/>
@@ -66,4 +60,10 @@
         <material name="red"/>
     </visual>
+    <collision>
+        <origin xyz="0 0 0.038" rpy="0 0 0"/>
+        <geometry>
+            <box size="0.263 0.31 0.04"/>
+        </geometry>
+    </collision>
 </link>
   <!-- Rear LEFT WHEEL -->
@@ -83,4 +83,9 @@
         <material name="blue"/>
     </visual>
+    <collision>
+        <geometry>
+            <cylinder length="0.04" radius="0.0485" />
+        </geometry>
+    </collision>
 </link>
   <!-- Rear RIGHT WHEEL -->
@@ -100,4 +105,9 @@
         <material name="blue"/>
     </visual>
+    <collision>
+        <geometry>
+            <cylinder length="0.04" radius="0.0485" />
+        </geometry>
+    </collision>
 </link>
 <!-- FRONT -->
@@ -133,4 +143,9 @@
         <material name="blue"/>
     </visual>
+    <collision>
+        <geometry>
+            <cylinder length="0.04" radius="0.0485" />
+        </geometry>
+    </collision>
 </link>
 <joint name="front_left_wheel_steer_joint" type="revolute">
@@ -138,5 +153,5 @@
     <axis xyz="0 0 1"/>
     <parent link="base_link"/>
-    <child link="front__left_wheel_steer"/>
+    <child link="front_left_wheel_steer"/>
     <origin rpy="0 0 0" xyz="0.360 0 0"/>
   </joint>
@@ -148,4 +163,9 @@
       <material name="black"/>
     </visual>
+    <collision>
+      <geometry>
+        <cylinder length="0.01" radius="0.01"/>
+      </geometry>
+    </collision>
   </link>
   <!-- FRONT RIGHT WHEEL -->
@@ -165,4 +185,9 @@
         <material name="blue"/>
     </visual>
+    <collision>
+        <geometry>
+            <cylinder length="0.04" radius="0.0485" />
+        </geometry>
+    </collision>
 </link>
 <joint name="front_right_wheel_steer_joint" type="revolute">
@@ -180,4 +205,9 @@
       <material name="black"/>
     </visual>
+    <collision>
+      <geometry>
+        <cylinder length="0.01" radius="0.01"/>
+      </geometry>
+    </collision>
   </link>
     </robot>
