Commit message: Update robot_core3.xacro

File: description/robot_core3.xacro (robot description, xacro)
@@ -1,5 +1,5 @@
 <?xml version="1.0"?>
 <robot xmlns:xacro="http://www.ros.org/wiki/xacro" >
-    <!-- <xacro:include filename="inertial_macros.xacro"/> -->
+    <xacro:include filename="inertial_macros.xacro"/>
     <material name="white">
         <color rgba="1 1 1 1" />
@@ -42,4 +42,7 @@
             </geometry>
         </collision>
+        <xacro:inertial_box mass="0.5" x="0.515" y="0.31" z="0.097">
+            <origin xyz="0.2575 0 0.0675" rpy="0 0 0"/>
+        </xacro:inertial_box>
     </link>
     <gazebo reference="chassis">
@@ -66,4 +69,7 @@
         </geometry>
     </collision>
+        <xacro:inertial_box mass="0.5" x="0.263" y="0.31" z="0.04">
+            <origin xyz="0 0 0.038" rpy="0 0 0"/>
+        </xacro:inertial_box>
 </link>
     <gazebo reference="upper_chassis">
@@ -79,4 +85,5 @@
     <axis xyz="0 0 1"/>
 </joint>
+<!--  -->
 <link name="rear_left_wheel">
     <visual>
@@ -86,10 +93,16 @@
         <material name="blue"/>
     </visual>
-    <collision>
-        <geometry>
-            <cylinder length="0.04" radius="0.0485" />
-        </geometry>
-    </collision>
-</link>
+<!--  -->
+    <collision>
+        <geometry>
+            <cylinder length="0.04" radius="0.0485" />
+        </geometry>
+    </collision>
+<!--  -->
+    <xacro:inertial_cylinder mass="0.1" length="0.04" radius="0.0485">
+            <origin xyz="0 0 0" rpy="0 0 0"/>
+        </xacro:inertial_cylinder>
+</link>
+<!--  -->
     <gazebo reference="rear_left_wheel">
         <material>Gazebo/Blue</material>
@@ -104,4 +117,5 @@
     <axis xyz="0 0 -1"/>
 </joint>
+<!--  -->
 <link name="rear_right_wheel">
     <visual>
@@ -111,9 +125,14 @@
         <material name="blue"/>
     </visual>
-    <collision>
-        <geometry>
-            <cylinder length="0.04" radius="0.0485" />
-        </geometry>
-    </collision>
+<!--  -->
+    <collision>
+        <geometry>
+            <cylinder length="0.04" radius="0.0485" />
+        </geometry>
+    </collision>
+<!--  -->
+        <xacro:inertial_cylinder mass="0.1" length="0.04" radius="0.0485">
+            <origin xyz="0 0 0" rpy="0 0 0"/>
+        </xacro:inertial_cylinder>
 </link>
     <gazebo reference="rear_right_wheel">
@@ -145,4 +164,5 @@
     <axis xyz="0 0 1"/>
 </joint>
+<!--  -->
 <link name="front_left_wheel">
     <visual>
@@ -152,13 +172,20 @@
         <material name="blue"/>
     </visual>
-    <collision>
-        <geometry>
-            <cylinder length="0.04" radius="0.0485" />
-        </geometry>
-    </collision>
-</link>
+<!--  -->
+    <collision>
+        <geometry>
+            <cylinder length="0.04" radius="0.0485" />
+        </geometry>
+    </collision>
+<!--  -->
+    <xacro:inertial_cylinder mass="0.1" length="0.04" radius="0.0485">
+            <origin xyz="0 0 0" rpy="0 0 0"/>
+    </xacro:inertial_cylinder>
+</link>
+<!--  -->
     <gazebo reference="front_left_wheel">
         <material>Gazebo/Blue</material>
     </gazebo>
+<!--  -->
 <joint name="front_left_wheel_steer_joint" type="revolute">
     <limit lower="-1" upper="1" effort="1" velocity="5"/>
@@ -168,4 +195,5 @@
     <origin rpy="0 0 0" xyz="0.360 0 0"/>
   </joint>
+<!--  -->
 <link name="front_left_wheel_steer">
     <visual>
@@ -175,10 +203,13 @@
       <material name="black"/>
     </visual>
-    <collision>
-      <geometry>
-        <cylinder length="0.01" radius="0.01"/>
-      </geometry>
-    </collision>
+<!--  -->
+    <collision>
+      <geometry>
+        <cylinder length="0.01" radius="0.01"/>
+      </geometry>
+    </collision>
+<!--  -->
   </link>
+<!--  -->
     <gazebo reference="front_left_wheel_steer">
         <material>Gazebo/Black</material>
@@ -193,4 +224,5 @@
     <axis xyz="0 0 -1"/>
 </joint>
+<!--  -->
 <link name="front_right_wheel">
     <visual>
@@ -200,10 +232,16 @@
         <material name="blue"/>
     </visual>
-    <collision>
-        <geometry>
-            <cylinder length="0.04" radius="0.0485" />
-        </geometry>
-    </collision>
-</link>
+<!--  -->
+    <collision>
+        <geometry>
+            <cylinder length="0.04" radius="0.0485" />
+        </geometry>
+    </collision>
+<!--  -->
+    <xacro:inertial_cylinder mass="0.1" length="0.04" radius="0.0485">
+            <origin xyz="0 0 0" rpy="0 0 0"/>
+    </xacro:inertial_cylinder>
+</link>
+<!--  -->
     <gazebo reference="front_right_wheel">
         <material>Gazebo/Blue</material>
@@ -229,4 +267,5 @@
     </collision>
   </link>
+<!--  -->
     <gazebo reference="front_right_wheel_steer">
         <material>Gazebo/Black</material>

Commit message: Update robot_core3.xacro

File: description/robot_core3.xacro (robot description, xacro)
@@ -105,5 +105,5 @@
 </link>
 <!--  -->
-    <gazebo reference="rear_left_wheel">
+    <gazebo reference="rear_left_joint">
         <material>Gazebo/Blue</material>
     </gazebo>
@@ -136,5 +136,5 @@
         </xacro:inertial_cylinder>
 </link>
-    <gazebo reference="rear_right_wheel">
+    <gazebo reference="rear_right_joint">
         <material>Gazebo/Blue</material>
     </gazebo>
@@ -184,5 +184,5 @@
 </link>
 <!--  -->
-    <gazebo reference="front_left_wheel">
+    <gazebo reference="front_left_joint">
         <material>Gazebo/Blue</material>
     </gazebo>
@@ -212,5 +212,5 @@
   </link>
 <!--  -->
-    <gazebo reference="front_left_wheel_steer">
+    <gazebo reference="left_steering_joint">
         <material>Gazebo/Black</material>
     </gazebo>
@@ -244,5 +244,5 @@
 </link>
 <!--  -->
-    <gazebo reference="front_right_wheel">
+    <gazebo reference="front_right_joint">
         <material>Gazebo/Blue</material>
     </gazebo>
@@ -268,6 +268,9 @@
   </link>
 <!--  -->
-    <gazebo reference="front_right_wheel_steer">
+    <gazebo reference="right_steering_joint">
         <material>Gazebo/Black</material>
     </gazebo>
+    <!-- <gazebo reference="steering_wheel_joint">
+        <material>Gazebo/Black</material>
+    </gazebo> -->
     </robot>
